File: eagle-cad/sensorboard.brd (EAGLE design)
At the start: 49.5 x 49.5 mm, 37 parts, among them IC1 MCP1702-33, U1 ATMEGA328P_PDIP, Y1 16MHz

Commit message: Fixed crystal cap values
Parts:
- C8, C9: value 0.1uF -> 22pF
Routing:
- added copper zone on layer 1, net GND
Other:
- board text added: "Sensor hub v1.8"
- board text removed: "Sensor hub v1.7"
Changed lines of the file:
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@@
 <?xml version="1.0" encoding="utf-8"?>
 <!DOCTYPE eagle SYSTEM "eagle.dtd">
-<eagle version="6.4">
+<eagle version="6.5.0">
 <drawing>
 <settings>
@@
 <board>
 <plain>
-<text x="39.37" y="25.4" size="1.27" layer="22" rot="MR90">Sensor hub v1.7</text>
+<text x="39.37" y="25.4" size="1.27" layer="22" rot="MR90">Sensor hub v1.8</text>
 <text x="36.195" y="25.4" size="1.27" layer="22" rot="MR90">Pertti Erkkilä 2013</text>
 <wire x1="2.54" y1="0" x2="46.99" y2="0" width="0" layer="20"/>
@@
 </class>
 </classes>
-<designrules name="ITEADstudio_DRC">
+<designrules name="LaenPCBOrder">
 <description language="de">&lt;b&gt;EAGLE Design Rules&lt;/b&gt;
 &lt;p&gt;
@@
 Einstellungen hier und speichern die Design Rules unter
 einem neuen Namen ab.</description>
-<description language="en">&lt;b&gt;iTead&lt;/b&gt;
+<description language="en">&lt;b&gt;Laen's PCB Order Design Rules&lt;/b&gt;
 &lt;p&gt;
-The default Design Rules have been set to cover
-a wide range of applications. Your particular design
-may have different requirements, so please make the
-necessary adjustments and save your customized
-design rules under a new name.</description>
-<description language="zh">&lt;b&gt;Seeed Studio EAGLE Design Rules&lt;/b&gt;
-</description>
+Please make sure your boards conform to these design rules.</description>
 <param name="layerSetup" value="(1*16)"/>
-<param name="mtCopper" value="0.035mm 0.035mm 0.035mm 0.035mm 0.035mm 0.035mm 0.035mm 0.035mm 0.035mm 0.035mm 0.035mm 0.035mm 0.035mm 0.035mm 0.035mm 0.035mm"/>
-<param name="mtIsolate" value="1.5mm 0.15mm 0.2mm 0.15mm 0.2mm 0.15mm 0.2mm 0.15mm 0.2mm 0.15mm 0.2mm 0.15mm 0.2mm 0.15mm 0.2mm"/>
+<param name="mtCopper" value="0.0356mm 0.0356mm 0.0356mm 0.0356mm 0.0356mm 0.0356mm 0.0356mm 0.0356mm 0.0356mm 0.0356mm 0.0356mm 0.0356mm 0.0356mm 0.0356mm 0.0356mm 0.0356mm"/>
+<param name="mtIsolate" value="1.5011mm 0.1499mm 0.2007mm 0.1499mm 0.2007mm 0.1499mm 0.2007mm 0.1499mm 0.2007mm 0.1499mm 0.2007mm 0.1499mm 0.2007mm 0.1499mm 0.2007mm"/>
 <param name="mdWireWire" value="6mil"/>
 <param name="mdWirePad" value="6mil"/>
@@
 <param name="mdPadVia" value="6mil"/>
 <param name="mdViaVia" value="6mil"/>
-<param name="mdSmdPad" value="0mil"/>
-<param name="mdSmdVia" value="0mil"/>
-<param name="mdSmdSmd" value="0mil"/>
+<param name="mdSmdPad" value="6mil"/>
+<param name="mdSmdVia" value="6mil"/>
+<param name="mdSmdSmd" value="6mil"/>
 <param name="mdViaViaSameLayer" value="8mil"/>
 <param name="mnLayersViaInSmd" value="2"/>
-<param name="mdCopperDimension" value="10mil"/>
-<param name="mdDrill" value="10mil"/>
+<param name="mdCopperDimension" value="15mil"/>
+<param name="mdDrill" value="6mil"/>
 <param name="mdSmdStop" value="0mil"/>
 <param name="msWidth" value="6mil"/>
-<param name="msDrill" value="12mil"/>
-<param name="msMicroVia" value="12mil"/>
+<param name="msDrill" value="13mil"/>
+<param name="msMicroVia" value="13mil"/>
 <param name="msBlindViaRatio" value="0.5"/>
 <param name="rvPadTop" value="0.25"/>
@@
 <param name="rvMicroViaOuter" value="0.25"/>
 <param name="rvMicroViaInner" value="0.25"/>
-<param name="rlMinPadTop" value="10mil"/>
+<param name="rlMinPadTop" value="7mil"/>
 <param name="rlMaxPadTop" value="20mil"/>
-<param name="rlMinPadInner" value="10mil"/>
+<param name="rlMinPadInner" value="7mil"/>
 <param name="rlMaxPadInner" value="20mil"/>
-<param name="rlMinPadBottom" value="10mil"/>
+<param name="rlMinPadBottom" value="7mil"/>
 <param name="rlMaxPadBottom" value="20mil"/>
-<param name="rlMinViaOuter" value="6mil"/>
+<param name="rlMinViaOuter" value="7mil"/>
 <param name="rlMaxViaOuter" value="20mil"/>
-<param name="rlMinViaInner" value="6mil"/>
+<param name="rlMinViaInner" value="7mil"/>
 <param name="rlMaxViaInner" value="20mil"/>
 <param name="rlMinMicroViaOuter" value="4mil"/>
@@
 <param name="psTop" value="-1"/>
 <param name="psBottom" value="-1"/>
-<param name="psFirst" value="0"/>
+<param name="psFirst" value="-1"/>
 <param name="psElongationLong" value="100"/>
 <param name="psElongationOffset" value="100"/>
 <param name="mvStopFrame" value="1"/>
 <param name="mvCreamFrame" value="0"/>
-<param name="mlMinStopFrame" value="2mil"/>
-<param name="mlMaxStopFrame" value="2mil"/>
+<param name="mlMinStopFrame" value="4mil"/>
+<param name="mlMaxStopFrame" value="4mil"/>
 <param name="mlMinCreamFrame" value="0mil"/>
 <param name="mlMaxCreamFrame" value="0mil"/>
-<param name="mlViaStopLimit" value="100mil"/>
+<param name="mlViaStopLimit" value="0mil"/>
 <param name="srRoundness" value="0"/>
 <param name="srMinRoundness" value="0mil"/>
@@
 <param name="checkAngle" value="0"/>
 <param name="checkFont" value="1"/>
-<param name="checkRestrict" value="0"/>
+<param name="checkRestrict" value="1"/>
 <param name="useDiameter" value="13"/>
 <param name="maxErrors" value="50"/>
@@
 <attribute name="VALUE" x="15.24" y="22.225" size="1.27" layer="27"/>
 </element>
-<element name="C8" library="SparkFun-Capacitors" package="CAP-PTH-SMALLEZ" value="0.1uF" x="33.02" y="6.35" smashed="yes" rot="R270">
+<element name="C8" library="SparkFun-Capacitors" package="CAP-PTH-SMALLEZ" value="22pF" x="33.02" y="6.35" smashed="yes" rot="R270">
 <attribute name="VALUE" x="30.48" y="7.62" size="0.6096" layer="27" rot="R270"/>
 </element>
-<element name="C9" library="SparkFun-Capacitors" package="CAP-PTH-SMALLEZ" value="0.1uF" x="30.48" y="6.35" smashed="yes" rot="R270">
+<element name="C9" library="SparkFun-Capacitors" package="CAP-PTH-SMALLEZ" value="22pF" x="30.48" y="6.35" smashed="yes" rot="R270">
 <attribute name="VALUE" x="27.94" y="7.62" size="0.6096" layer="27" rot="R270"/>
 </element>
@@
 </polygon>
 <contactref element="VCC-" pad="1"/>
+<polygon width="0.6096" layer="1" isolate="0.4064">
+<vertex x="-2.54" y="52.07"/>
+<vertex x="52.07" y="52.07"/>
+<vertex x="52.07" y="-2.54"/>
+<vertex x="-2.54" y="-2.54"/>
+</polygon>
 </signal>
 <signal name="N$7">

Commit message: Fixed resistor divider cap value
Parts:
- C6: value 1uF -> 0.1uF
Changed lines of the file:
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@@
 <attribute name="VALUE" x="22.86" y="3.302" size="1.016" layer="21" font="vector" ratio="15"/>
 </element>
-<element name="C6" library="SparkFun-Capacitors" package="CAP-PTH-SMALLEZ" value="1uF" x="20.32" y="6.35" smashed="yes">
+<element name="C6" library="SparkFun-Capacitors" package="CAP-PTH-SMALLEZ" value="0.1uF" x="20.32" y="6.35" smashed="yes">
 <attribute name="VALUE" x="19.05" y="3.81" size="0.6096" layer="27"/>
 </element>
